File: 8 step sequencer/CAD/PCB/8 Steps/8steps.sch (EAGLE design)
At the start: 30 parts, among them IC1 4040N, IC2 4040N, IC3 7805TV, IC4 4051N, IC5 4051N, IC6 LM324N

Commit message: new fabrication files of  8 steps
Parts:
- added JP10: PWR, pinhead:PINHD-1X2
- added PAD1, PAD2, PAD3: WIREPADSMD1,27-254, wirepad:WIREPADSMD1,27-254
Connections:
- net B0: now also PAD1.P
- net B1: now also PAD2.P
- net B2: now also PAD3.P
- net GND: now also JP10.1
- net V5V: now also JP10.2
Other:
- note added: "C"
Changed lines of the file:
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@@
 <part name="C2" library="rcl" deviceset="CPOL-EU" device="E2.5-7" value="100u"/>
 <part name="P+2" library="supply1" deviceset="VCC" device=""/>
+<part name="JP10" library="pinhead" deviceset="PINHD-1X2" device="" value="PWR"/>
+<part name="GND14" library="supply1" deviceset="GND" device=""/>
+<part name="PAD1" library="wirepad" deviceset="WIREPAD" device="SMD1,27-254" value=""/>
+<part name="PAD2" library="wirepad" deviceset="WIREPAD" device="SMD1,27-254" value=""/>
+<part name="PAD3" library="wirepad" deviceset="WIREPAD" device="SMD1,27-254" value=""/>
 </parts>
 <sheets>
@@
 <text x="205.74" y="162.56" size="1.778" layer="97">GATE/LED </text>
 <text x="205.74" y="88.9" size="1.778" layer="97">CV</text>
+<text x="256.54" y="7.62" size="2.54" layer="94">C</text>
 </plain>
 <instances>
@@
 <instance part="P+2" gate="VCC" x="27.94" y="109.22" rot="R90"/>
 <instance part="IC6" gate="P" x="66.04" y="30.48"/>
+<instance part="JP10" gate="G$1" x="111.76" y="101.6" rot="R180"/>
+<instance part="GND14" gate="1" x="121.92" y="93.98"/>
+<instance part="PAD1" gate="G$1" x="139.7" y="119.38"/>
+<instance part="PAD2" gate="G$1" x="139.7" y="114.3"/>
+<instance part="PAD3" gate="G$1" x="139.7" y="109.22"/>
 </instances>
 <busses>
@@
 <junction x="20.32" y="20.32"/>
 </segment>
+<segment>
+<pinref part="JP10" gate="G$1" pin="1"/>
+<pinref part="GND14" gate="1" pin="GND"/>
+<wire x1="114.3" y1="99.06" x2="121.92" y2="99.06" width="0.1524" layer="91"/>
+<wire x1="121.92" y1="99.06" x2="121.92" y2="96.52" width="0.1524" layer="91"/>
+</segment>
 </net>
 <net name="VCC" class="0">
@@
 <wire x1="35.56" y1="157.48" x2="22.86" y2="157.48" width="0.1524" layer="91"/>
 </segment>
+<segment>
+<pinref part="PAD1" gate="G$1" pin="P"/>
+<wire x1="142.24" y1="119.38" x2="149.86" y2="119.38" width="0.1524" layer="91"/>
+<label x="147.32" y="119.38" size="2.54" layer="95"/>
+</segment>
 </net>
 <net name="B1" class="0">
@@
 <wire x1="35.56" y1="154.94" x2="22.86" y2="154.94" width="0.1524" layer="91"/>
 </segment>
+<segment>
+<pinref part="PAD2" gate="G$1" pin="P"/>
+<wire x1="142.24" y1="114.3" x2="149.86" y2="114.3" width="0.1524" layer="91"/>
+<label x="147.32" y="114.3" size="2.54" layer="95"/>
+</segment>
 </net>
 <net name="B2" class="0">
@@
 <pinref part="IC1" gate="A" pin="Q3"/>
 <wire x1="35.56" y1="152.4" x2="22.86" y2="152.4" width="0.1524" layer="91"/>
+</segment>
+<segment>
+<pinref part="PAD3" gate="G$1" pin="P"/>
+<wire x1="142.24" y1="109.22" x2="149.86" y2="109.22" width="0.1524" layer="91"/>
+<label x="147.32" y="109.22" size="2.54" layer="95"/>
 </segment>
 </net>
@@
 <junction x="152.4" y="38.1"/>
 </segment>
-</net>
+<segment>
+<pinref part="JP10" gate="G$1" pin="2"/>
+<wire x1="114.3" y1="101.6" x2="124.46" y2="101.6" width="0.1524" layer="91"/>
+<label x="119.38" y="101.6" size="1.778" layer="95"/>
+</segment>
+</net>
